File: WindTunnel/wiring-diagram/wiring-diagram.kicad_sch (KiCad schematic)
At the start: 7 parts, among them J1 Barrel_Jack, M1 Stepper_Motor_bipolar, SW1 SW_SPST, SW2 LIMIT SW

Commit message: final wiring diagram
Parts:
- added U4: ~, symbol my-wiring-symbols:motor-conn
Connections:
- net at U2.10 (A+): now also U4.; no longer M1.4
- net at U2.7 (B-): now also U4.; no longer M1.2 (-)
- net at U2.8 (B+): now also U4.; no longer M1.1
- net at U2.9 (A-): now also U4.; no longer M1.3
- new net: M1.1, U4.
- new net: M1.2 (-), U4.
- new net: M1.3, U4.
- new net: M1.4, U4.
Other:
- note added: "16 AWG"
- note added: "22 AWG"
- note added: "Motor Connector (what type?)"
- note added: "Wire Sizes"
- moved on the sheet: J1, M1
